File: nascontrol-remote.kicad_sch (KiCad schematic)
At the start: 22 parts, among them J101 Serial, J102 System IN, J103 Control, J104 System OUT, U101 EL817, U102 EL817, U103 EL817, U104 EL817

Commit message: Fix PWR and RST issue
Signed-off-by: Benedikt Spranger <b.spranger@linutronix.de>
Connections:
- net ~{PWRBTN1} is gone; now on net GND: J102.6 (Pin_6)
- net ~{RST1} is gone; now on net ~{RST2}: J102.7 (Pin_7)
- net GND: now also J102.10 (Pin_10), J104.10 (Pin_10), J104.6 (Pin_6); no longer J102.8 (Pin_8), J104.3 (Pin_3), J104.4 (Pin_4), J104.8 (Pin_8)
- net HDDLED: no longer R102.1
- net HDLED1+: now also J104.1 (Pin_1)
- net HDLED1-: now also J104.3 (Pin_3)
- net PLED1+: now also J104.2 (Pin_2)
- net PLED1-: now also J104.4 (Pin_4)
- net PWR: now also R102.1
- net PWRLED: no longer R104.1
- net RST: now also R104.1
- net ~{PWRBTN2}: now also J102.8 (Pin_8), J104.8 (Pin_8), R101.1, U101.4; no longer J104.6 (Pin_6)
- net ~{RST2}: now also R103.1, U102.4
- removed net HDLED2+: J104.1 (Pin_1), R101.1, U101.4
- removed net PLED2+: J104.2 (Pin_2), R103.1, U102.4
- no-connect marks 8 -> 6
Changed lines of the file:
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@@
     (comment 4 "This work is licensed under the CERN-OHL-S v2")
   )
-  (junction (at 118.11 129.54) (diameter 0) (color 0 0 0 0)
-  )
   (junction (at 68.58 88.9) (diameter 0) (color 0 0 0 0)
   )
@@
   (junction (at 182.88 119.38) (diameter 0) (color 0 0 0 0)
   )
+  (junction (at 135.89 96.52) (diameter 0) (color 0 0 0 0)
+  )
   (junction (at 68.58 165.1) (diameter 0) (color 0 0 0 0)
   )
@@
   (junction (at 198.12 129.54) (diameter 0) (color 0 0 0 0)
   )
-  (junction (at 135.89 132.08) (diameter 0) (color 0 0 0 0)
+  (junction (at 135.89 134.62) (diameter 0) (color 0 0 0 0)
   )
   (junction (at 210.82 109.22) (diameter 0) (color 0 0 0 0)
   )
-  (no_connect (at 133.35 134.62))
-  (no_connect (at 133.35 96.52))
   (no_connect (at 120.65 60.96))
   (no_connect (at 133.35 60.96))
@@
   (no_connect (at 133.35 53.34))
   (no_connect (at 120.65 50.8))
+  (wire (pts (xy 135.89 134.62) (xy 135.89 137.16))
+    (stroke (width 0) (type default))
+  )
   (wire (pts (xy 68.58 127) (xy 68.58 124.46))
     (stroke (width 0) (type default))
@@
     (stroke (width 0) (type default))
   )
+  (wire (pts (xy 135.89 91.44) (xy 135.89 96.52))
+    (stroke (width 0) (type default))
+  )
   (wire (pts (xy 68.58 38.1) (xy 68.58 40.64))
     (stroke (width 0) (type default))
@@
     (stroke (width 0) (type default))
   )
-  (wire (pts (xy 135.89 137.16) (xy 135.89 132.08))
-    (stroke (width 0) (type default))
-  )
   (wire (pts (xy 66.04 50.8) (xy 68.58 50.8))
     (stroke (width 0) (type default))
@@
     (stroke (width 0) (type default))
   )
-  (wire (pts (xy 118.11 127) (xy 118.11 129.54))
-    (stroke (width 0) (type default))
-  )
   (wire (pts (xy 208.28 111.76) (xy 213.36 111.76))
     (stroke (width 0) (type default))
   )
+  (wire (pts (xy 135.89 96.52) (xy 135.89 99.06))
+    (stroke (width 0) (type default))
+  )
   (wire (pts (xy 187.96 129.54) (xy 198.12 129.54))
     (stroke (width 0) (type default))
@@
     (stroke (width 0) (type default))
   )
+  (wire (pts (xy 135.89 129.54) (xy 135.89 134.62))
+    (stroke (width 0) (type default))
+  )
   (wire (pts (xy 187.96 53.34) (xy 190.5 53.34))
     (stroke (width 0) (type default))
@@
     (stroke (width 0) (type default))
   )
-  (wire (pts (xy 133.35 129.54) (xy 138.43 129.54))
-    (stroke (width 0) (type default))
-  )
   (wire (pts (xy 48.26 93.98) (xy 50.8 93.98))
     (stroke (width 0) (type default))
@@
     (stroke (width 0) (type default))
   )
+  (wire (pts (xy 133.35 134.62) (xy 135.89 134.62))
+    (stroke (width 0) (type default))
+  )
   (wire (pts (xy 68.58 50.8) (xy 68.58 48.26))
     (stroke (width 0) (type default))
@@
     (stroke (width 0) (type default))
   )
+  (wire (pts (xy 133.35 132.08) (xy 138.43 132.08))
+    (stroke (width 0) (type default))
+  )
+  (wire (pts (xy 133.35 93.98) (xy 138.43 93.98))
+    (stroke (width 0) (type default))
+  )
   (wire (pts (xy 210.82 109.22) (xy 213.36 109.22))
     (stroke (width 0) (type default))
@@
     (stroke (width 0) (type default))
   )
-  (wire (pts (xy 135.89 132.08) (xy 133.35 132.08))
-    (stroke (width 0) (type default))
-  )
   (wire (pts (xy 198.12 127) (xy 198.12 129.54))
     (stroke (width 0) (type default))
@@
     (stroke (width 0) (type default))
   )
-  (wire (pts (xy 133.35 88.9) (xy 135.89 88.9))
-    (stroke (width 0) (type default))
-  )
-  (wire (pts (xy 135.89 93.98) (xy 133.35 93.98))
+  (wire (pts (xy 133.35 88.9) (xy 138.43 88.9))
     (stroke (width 0) (type default))
   )
@@
     (stroke (width 0) (type default))
   )
-  (wire (pts (xy 135.89 99.06) (xy 135.89 93.98))
-    (stroke (width 0) (type default))
-  )
   (wire (pts (xy 118.11 96.52) (xy 118.11 99.06))
     (stroke (width 0) (type default))
   )
+  (wire (pts (xy 133.35 129.54) (xy 135.89 129.54))
+    (stroke (width 0) (type default))
+  )
   (wire (pts (xy 208.28 114.3) (xy 213.36 114.3))
     (stroke (width 0) (type default))
   )
-  (wire (pts (xy 133.35 127) (xy 135.89 127))
+  (wire (pts (xy 133.35 127) (xy 138.43 127))
     (stroke (width 0) (type default))
   )
@@
     (stroke (width 0) (type default))
   )
-  (wire (pts (xy 135.89 127) (xy 135.89 132.08))
-    (stroke (width 0) (type default))
-  )
   (wire (pts (xy 48.26 88.9) (xy 50.8 88.9))
     (stroke (width 0) (type default))
@@
     (stroke (width 0) (type default))
   )
+  (wire (pts (xy 133.35 96.52) (xy 135.89 96.52))
+    (stroke (width 0) (type default))
+  )
   (wire (pts (xy 66.04 132.08) (xy 68.58 132.08))
     (stroke (width 0) (type default))
   )
-  (wire (pts (xy 118.11 127) (xy 120.65 127))
+  (wire (pts (xy 115.57 127) (xy 120.65 127))
     (stroke (width 0) (type default))
   )
@@
     (stroke (width 0) (type default))
   )
-  (wire (pts (xy 133.35 86.36) (xy 135.89 86.36))
+  (wire (pts (xy 133.35 86.36) (xy 138.43 86.36))
     (stroke (width 0) (type default))
   )
@@
     (stroke (width 0) (type default))
   )
-  (text "Remove\nPin" (at 133.35 96.52 90)
-    (effects (font (size 1.27 1.27)) (justify right bottom))
-  )
-  (text "Remove\nPin" (at 133.35 134.62 90)
-    (effects (font (size 1.27 1.27)) (justify right bottom))
-  )
   (text "Remove\nPin" (at 133.35 60.96 90)
     (effects (font (size 1.27 1.27)) (justify right bottom))
   )
-  (label "PWRLED" (at 38.1 88.9 180) (fields_autoplaced)
-    (effects (font (size 1.27 1.27)) (justify right bottom))
-  )
-  (label "PLED2+" (at 138.43 124.46 0) (fields_autoplaced)
+  (label "~{PWRBTN2}" (at 138.43 93.98 0) (fields_autoplaced)
     (effects (font (size 1.27 1.27)) (justify left bottom))
   )
@@
     (effects (font (size 1.27 1.27)) (justify left bottom))
   )
-  (label "PLED1-" (at 135.89 88.9 0) (fields_autoplaced)
+  (label "PLED1-" (at 138.43 88.9 0) (fields_autoplaced)
+    (effects (font (size 1.27 1.27)) (justify left bottom))
+  )
+  (label "RST" (at 38.1 88.9 180) (fields_autoplaced)
+    (effects (font (size 1.27 1.27)) (justify right bottom))
+  )
+  (label "~{PWRBTN2}" (at 71.12 50.8 0) (fields_autoplaced)
     (effects (font (size 1.27 1.27)) (justify left bottom))
   )
@@
     (effects (font (size 1.27 1.27)) (justify right bottom))
   )
-  (label "~{PWRBTN1}" (at 135.89 91.44 0) (fields_autoplaced)
-    (effects (font (size 1.27 1.27)) (justify left bottom))
-  )
   (label "PWRLED" (at 213.36 104.14 0) (fields_autoplaced)
     (effects (font (size 1.27 1.27)) (justify left bottom))
@@
     (effects (font (size 1.27 1.27)) (justify left bottom))
   )
+  (label "~{RST2}" (at 115.57 93.98 180) (fields_autoplaced)
+    (effects (font (size 1.27 1.27)) (justify right bottom))
+  )
   (label "PLED1-" (at 48.26 170.18 180) (fields_autoplaced)
     (effects (font (size 1.27 1.27)) (justify right bottom))
   )
-  (label "PLED1+" (at 135.89 86.36 0) (fields_autoplaced)
+  (label "PLED1+" (at 138.43 86.36 0) (fields_autoplaced)
     (effects (font (size 1.27 1.27)) (justify left bottom))
   )
@@
     (effects (font (size 1.27 1.27)) (justify right bottom))
   )
+  (label "PLED1+" (at 138.43 124.46 0) (fields_autoplaced)
+    (effects (font (size 1.27 1.27)) (justify left bottom))
+  )
+  (label "PLED1-" (at 138.43 127 0) (fields_autoplaced)
+    (effects (font (size 1.27 1.27)) (justify left bottom))
+  )
   (label "RX" (at 187.96 60.96 180) (fields_autoplaced)
     (effects (font (size 1.27 1.27)) (justify right bottom))
   )
-  (label "HDLED2+" (at 71.12 50.8 0) (fields_autoplaced)
-    (effects (font (size 1.27 1.27)) (justify left bottom))
-  )
   (label "HDDLED" (at 213.36 106.68 0) (fields_autoplaced)
     (effects (font (size 1.27 1.27)) (justify left bottom))
   )
+  (label "PWR" (at 38.1 50.8 180) (fields_autoplaced)
+    (effects (font (size 1.27 1.27)) (justify right bottom))
+  )
   (label "HDLED1+" (at 38.1 127 180) (fields_autoplaced)
     (effects (font (size 1.27 1.27)) (justify right bottom))
   )
-  (label "HDDLED" (at 38.1 50.8 180) (fields_autoplaced)
-    (effects (font (size 1.27 1.27)) (justify right bottom))
-  )
   (label "RTS" (at 187.96 66.04 180) (fields_autoplaced)
     (effects (font (size 1.27 1.27)) (justify right bottom))
@@
     (effects (font (size 1.27 1.27)) (justify left bottom))
   )
+  (label "~{RST2}" (at 71.12 88.9 0) (fields_autoplaced)
+    (effects (font (size 1.27 1.27)) (justify left bottom))
+  )
   (label "RST" (at 213.36 119.38 0) (fields_autoplaced)
     (effects (font (size 1.27 1.27)) (justify left bottom))
   )
-  (label "HDLED2+" (at 115.57 124.46 180) (fields_autoplaced)
-    (effects (font (size 1.27 1.27)) (justify right bottom))
-  )
   (label "A" (at 187.96 53.34 180) (fields_autoplaced)
     (effects (font (size 1.27 1.27)) (justify right bottom))
@@
     (effects (font (size 1.27 1.27)) (justify right bottom))
   )
+  (label "HDLED1+" (at 115.57 124.46 180) (fields_autoplaced)
+    (effects (font (size 1.27 1.27)) (justify right bottom))
+  )
   (label "PWR" (at 213.36 121.92 0) (fields_autoplaced)
     (effects (font (size 1.27 1.27)) (justify left bottom))
@@
     (effects (font (size 1.27 1.27)) (justify right bottom))
   )
-  (label "~{PWRBTN2}" (at 138.43 129.54 0) (fields_autoplaced)
-    (effects (font (size 1.27 1.27)) (justify left bottom))
-  )
-  (label "PLED2+" (at 71.12 88.9 0) (fields_autoplaced)
-    (effects (font (size 1.27 1.27)) (justify left bottom))
-  )
-  (label "~{RST1}" (at 115.57 93.98 180) (fields_autoplaced)
-    (effects (font (size 1.27 1.27)) (justify right bottom))
-  )
+  (label "~{PWRBTN2}" (at 138.43 132.08 0) (fields_autoplaced)
+    (effects (font (size 1.27 1.27)) (justify left bottom))
+  )
+  (label "HDLED1-" (at 115.57 127 180) (fields_autoplaced)
+    (effects (font (size 1.27 1.27)) (justify right bottom))
+  )

Commit message: Insulation cleanup
Signed-off-by: Benedikt Spranger <b.spranger@linutronix.de>
Parts:
- removed H101: ~, MountingHole:MountingHole_3.2mm_M3, symbol Mechanical:MountingHole
- added H101: ~, MountingHole:MountingHole_3.2mm_M3_Pad, symbol Mechanical:MountingHole_Pad
Connections:
- net GND: now also H101.1
Changed lines of the file:
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@@
+    (stroke (width 0) (type default))
+  )
+  (wire (pts (xy 241.3 139.7) (xy 241.3 142.24))
     (stroke (width 0) (type default))
   )
@@
     )
   )
-  (symbol (lib_id "Mechanical:MountingHole") (at 241.3 137.16 0) (unit 1)
-    (in_bom yes) (on_board yes) (dnp no) (fields_autoplaced)
-    (property "Reference" "H101" (at 243.84 134.6199 0)
-      (effects (font (size 1.27 1.27)) (justify left))
-    )
-    (property "Value" "~" (at 243.84 137.1599 0)
-      (effects (font (size 1.27 1.27)) (justify left))
-    )
-    (property "Footprint" "MountingHole:MountingHole_3.2mm_M3" (at 241.3 137.16 0)
-      (effects (font (size 1.27 1.27)) hide)
-    )
-    (property "Datasheet" "~" (at 241.3 137.16 0)
-      (effects (font (size 1.27 1.27)) hide)
-    )
-    (property "Description" "Mounting Hole M3" (at 241.3 137.16 0)
-      (effects (font (size 1.27 1.27)) hide)
-    )
-    (property "Manufacture" "N/A" (at 241.3 137.16 0)
-      (effects (font (size 1.27 1.27)) hide)
-    )
-    (property "assemble" "n" (at 241.3 137.16 0)
-      (effects (font (size 1.27 1.27)) hide)
-    )
-    (property "mpn" "N/A" (at 241.3 137.16 0)
-      (effects (font (size 1.27 1.27)) hide)
-    )
-    (instances
-      (project "nascontrol-remote"
-        (path "/a4396576-4100-4996-96eb-11896006f014"
-          (reference "H101") (unit 1)
-        )
-      )
-    )
-  )
   (symbol (lib_id "Isolator:EL817") (at 58.42 53.34 0) (unit 1)
     (in_bom yes) (on_board yes) (dnp no) (fields_autoplaced)
@@
     )
   )
+  (symbol (lib_id "Mechanical:MountingHole_Pad") (at 241.3 137.16 0) (unit 1)
+    (in_bom yes) (on_board yes) (dnp no) (fields_autoplaced)
+    (property "Reference" "H101" (at 243.84 134.6199 0)
+      (effects (font (size 1.27 1.27)) (justify left))
+    )
+    (property "Value" "~" (at 243.84 137.1599 0)
+      (effects (font (size 1.27 1.27)) (justify left))
+    )
+    (property "Footprint" "MountingHole:MountingHole_3.2mm_M3_Pad" (at 241.3 137.16 0)
+      (effects (font (size 1.27 1.27)) hide)
+    )
+    (property "Datasheet" "~" (at 241.3 137.16 0)
+      (effects (font (size 1.27 1.27)) hide)
+    )
+    (property "Description" "Mounting Hole M3" (at 241.3 137.16 0)
+      (effects (font (size 1.27 1.27)) hide)
+    )
+    (property "Manufacture" "N/A" (at 241.3 137.16 0)
+      (effects (font (size 1.27 1.27)) hide)
+    )
+    (property "assemble" "n" (at 241.3 137.16 0)
+      (effects (font (size 1.27 1.27)) hide)
+    )
+    (property "mpn" "N/A" (at 241.3 137.16 0)
+      (effects (font (size 1.27 1.27)) hide)
+    )
+    (pin "1")
+    (instances
+      (project "nascontrol-remote"
+        (path "/a4396576-4100-4996-96eb-11896006f014"
+          (reference "H101") (unit 1)
+        )
+      )
+    )
+  )
   (symbol (lib_id "power:+3V3") (at 68.58 152.4 0) (unit 1)
     (in_bom yes) (on_board yes) (dnp no) (fields_autoplaced)
@@
         )
       )
+    )
+  )
+  (symbol (lib_id "power:GND") (at 241.3 142.24 0) (mirror y) (unit 1)
+    (in_bom yes) (on_board yes) (dnp no) (fields_autoplaced)
+    (property "Reference" "#PWR0122" (at 241.3 148.59 0)
+      (effects (font (size 1.27 1.27)) hide)
+    )
+    (property "Value" "GND" (at 241.3 147.32 0)
+      (effects (font (size 1.27 1.27)))
+    )
+    (property "Footprint" "" (at 241.3 142.24 0)
+      (effects (font (size 1.27 1.27)) hide)
+    )
+    (property "Datasheet" "" (at 241.3 142.24 0)
+      (effects (font (size 1.27 1.27)) hide)
+    )
+    (pin "1")
+    (instances
+      (project "nascontrol-remote"
+        (path "/a4396576-4100-4996-96eb-11896006f014"
+          (reference "#PWR0122") (unit 1)
+        )
+      )
